Commit message: some changes

File: roboverse_data/assets/humanoidbench/table/urdf/table.urdf (robot description, URDF)
Before this commit: robot table, 1 links, 0 joints
Links:
- added link dummy_base
- link base_link: geometry collision box size=0.05 0.05 0.75; collision box size=0.05 0.05 0.75
Joints:
- added joint root_joint: type fixed, parent dummy_base, child base_link
