Commit message: fixed genesis to work with robot(collapse_fixed_joint false, fix_base_link false)

File: roboverse_data/robots/g1/urdf/g1_mygym_with_world.urdf (robot description, URDF)
Before this commit: robot g1_29dof_with_hand_rev_1_0, 54 links, 53 joints
Links:
- added link world
Joints:
- added joint base_to_world: type fixed, parent world, child pelvis
- joint pelvis_contour_joint: child pelvis -> pelvis_contour_link; parent pelvis_contour_link -> pelvis
