Commit message: new reward ro rech pos ori

File: roboverse_data/robots/g1/urdf/g1_mygym_for_reach.urdf (robot description, URDF)
Before this commit: robot g1_29dof_with_hand_rev_1_0, 54 links, 53 joints
Joints:
- joint right_elbow_joint: limit lower=-1.0472 upper=2.0944 effort=25 velocity=37 -> lower=-1.0472 upper=2.0944 effort=100 velocity=37
- joint right_shoulder_pitch_joint: limit lower=-3.0892 upper=2.6704 effort=25 velocity=37 -> lower=-3.0892 upper=2.6704 effort=50 velocity=37
- joint right_shoulder_roll_joint: limit lower=-2.2515 upper=1.5882 effort=25 velocity=37 -> lower=-2.2515 upper=1.5882 effort=100 velocity=37
- joint right_shoulder_yaw_joint: limit lower=-2.618 upper=2.618 effort=25 velocity=37 -> lower=-2.618 upper=2.618 effort=100 velocity=37
- joint right_wrist_pitch_joint: limit lower=-1.614429558 upper=1.614429558 effort=5 velocity=22 -> lower=-1.614429558 upper=1.614429558 effort=100 velocity=22
- joint right_wrist_roll_joint: limit lower=-1.972222054 upper=1.972222054 effort=25 velocity=37 -> lower=-1.972222054 upper=1.972222054 effort=100 velocity=37
- joint right_wrist_yaw_joint: limit lower=-1.614429558 upper=1.614429558 effort=5 velocity=22 -> lower=-1.614429558 upper=1.614429558 effort=100 velocity=22

Commit message: finally fix reach pos ori in genesis i hope

File: roboverse_data/robots/g1/urdf/g1_mygym_for_reach.urdf (robot description, URDF)
Before this commit: robot g1_29dof_with_hand_rev_1_0, 54 links, 53 joints
Links:
- link right_wrist_roll_link: geometry visual mesh filename=meshes/right_wrist_roll_link.STL
