Commit message: some fix in reward function

File: roboverse_data/robots/g1/urdf/g1_mygym_rotslide.urdf (robot description, URDF)
Before this commit: robot g1_29dof_with_hand_rev_1_0, 65 links, 64 joints
Joints:
- joint baseslide_joint2: limit lower=-5.5 upper=5.5 effort=300 velocity=0.05 -> lower=-2.0 upper=0.1 effort=30 velocity=0.05
