Commit message: automatic run ppo dagger grpo

File: roboverse_data/robots/g1/urdf/g1_mygym_rotslide.urdf (robot description, URDF)
Before this commit: robot g1_29dof_with_hand_rev_1_0, 65 links, 64 joints
Joints:
- joint waist_pitch_joint: type revolute -> fixed
- joint waist_roll_joint: type revolute -> fixed
- joint waist_yaw_joint: type revolute -> fixed
