Commit message: fix bug chairman simple

File: roboverse_data/robots/g1/urdf/g1_mygym_rotslide_simple.urdf (robot description, URDF)
Before this commit: robot g1_29dof_with_hand_rev_1_0, 65 links, 64 joints
Joints:
- joint baseslide_joint2: limit lower=-2.0 upper=0.1 effort=30 velocity=0.05 -> lower=-1.6 upper=0.1 effort=10 velocity=0.25

Commit message: worknig teacher i hope

File: roboverse_data/robots/g1/urdf/g1_mygym_rotslide_simple.urdf (robot description, URDF)
Before this commit: robot g1_29dof_with_hand_rev_1_0, 65 links, 64 joints
Joints:
- joint baseslide_joint: limit lower=-1.5 upper=1.5 effort=300 velocity=0.05 -> lower=-1.5 upper=1.5 effort=100 velocity=0.05
- joint baseslide_joint2: limit lower=-1.6 upper=0.1 effort=10 velocity=0.25 -> lower=-1.6 upper=0.1 effort=100 velocity=0.25
