Commit message: chairman with walking policy.pt  still not work well

File: roboverse_data/robots/g1/urdf/g1_mygym.urdf (robot description, URDF)
Before this commit: robot g1_29dof_with_hand_rev_1_0, 54 links, 53 joints
Links:
- added link ee_x_axis; visual cylinder length=0.06 radius=0.002
- added link ee_y_axis; visual cylinder length=0.06 radius=0.002
- added link ee_z_axis; visual cylinder length=0.06 radius=0.002
- added link left_ee_x_axis; visual cylinder length=0.06 radius=0.002
- added link left_ee_y_axis; visual cylinder length=0.06 radius=0.002
- added link left_ee_z_axis; visual cylinder length=0.06 radius=0.002
- added link left_endeffector; visual sphere radius=0.005
- link endeffector: mass 0.0000332 -> None; geometry visual sphere radius=0.005
Joints:
- added joint ee_x_axis_joint: type fixed, parent right_hand_palm_link, child ee_x_axis, origin xyz=0.07 0.07 0.0 rpy=-1.57 -1.57 0
- added joint ee_y_axis_joint: type fixed, parent right_hand_palm_link, child ee_y_axis, origin xyz=0.07 0.07 0.0 rpy=-1.57 -1.57 0
- added joint ee_z_axis_joint: type fixed, parent right_hand_palm_link, child ee_z_axis, origin xyz=0.07 0.07 0.0 rpy=-1.57 -1.57 0
- added joint left_ee_x_axis_joint: type fixed, parent left_hand_palm_link, child left_ee_x_axis, origin xyz=0.07 -0.07 0.0 rpy=-1.57 -1.57 0
- added joint left_ee_y_axis_joint: type fixed, parent left_hand_palm_link, child left_ee_y_axis, origin xyz=0.07 -0.07 0.0 rpy=-1.57 -1.57 0
- added joint left_ee_z_axis_joint: type fixed, parent left_hand_palm_link, child left_ee_z_axis, origin xyz=0.07 -0.07 0.0 rpy=-1.57 -1.57 0
- added joint left_endeffector_joint: type fixed, parent left_hand_palm_link, child left_endeffector, origin xyz=0.07 -0.07 0.0 rpy=-1.57 0 0

File: roboverse_data/robots/g1/urdf/g1_mygym_with_world.urdf (robot description, URDF)
Before this commit: robot g1_29dof_with_hand_rev_1_0, 55 links, 54 joints
Links:
- added link ee_x_axis; visual cylinder length=0.06 radius=0.002
- added link ee_y_axis; visual cylinder length=0.06 radius=0.002
- added link ee_z_axis; visual cylinder length=0.06 radius=0.002
- added link left_ee_x_axis; visual cylinder length=0.06 radius=0.002
- added link left_ee_y_axis; visual cylinder length=0.06 radius=0.002
- added link left_ee_z_axis; visual cylinder length=0.06 radius=0.002
- added link left_endeffector; visual sphere radius=0.005
- link endeffector: mass 0.0000332 -> None; geometry visual sphere radius=0.005
Joints:
- added joint ee_x_axis_joint: type fixed, parent right_hand_palm_link, child ee_x_axis, origin xyz=0.07 0.07 0.0 rpy=-1.57 -1.57 0
- added joint ee_y_axis_joint: type fixed, parent right_hand_palm_link, child ee_y_axis, origin xyz=0.07 0.07 0.0 rpy=-1.57 -1.57 0
- added joint ee_z_axis_joint: type fixed, parent right_hand_palm_link, child ee_z_axis, origin xyz=0.07 0.07 0.0 rpy=-1.57 -1.57 0
- added joint left_ee_x_axis_joint: type fixed, parent left_hand_palm_link, child left_ee_x_axis, origin xyz=0.07 -0.07 0.0 rpy=-1.57 -1.57 0
- added joint left_ee_y_axis_joint: type fixed, parent left_hand_palm_link, child left_ee_y_axis, origin xyz=0.07 -0.07 0.0 rpy=-1.57 -1.57 0
- added joint left_ee_z_axis_joint: type fixed, parent left_hand_palm_link, child left_ee_z_axis, origin xyz=0.07 -0.07 0.0 rpy=-1.57 -1.57 0
- added joint left_endeffector_joint: type fixed, parent left_hand_palm_link, child left_endeffector, origin xyz=0.07 -0.07 0.0 rpy=-1.57 0 0

Commit message: requirement3.yml added

File: roboverse_data/robots/g1/urdf/g1_mygym.urdf (robot description, URDF)
Before this commit: robot g1_29dof_with_hand_rev_1_0, 61 links, 60 joints
Links:
- removed link left_ee_x_axis
- removed link left_ee_y_axis
- removed link left_ee_z_axis
- removed link left_endeffector
Joints:
- removed joint left_ee_x_axis_joint
- removed joint left_ee_y_axis_joint
- removed joint left_ee_z_axis_joint
- removed joint left_endeffector_joint

Commit message: train

File: roboverse_data/robots/g1/urdf/g1_mygym.urdf (robot description, URDF)
Before this commit: robot g1_29dof_with_hand_rev_1_0, 57 links, 56 joints
Links:
- added link left_ee_x_axis; visual cylinder length=0.06 radius=0.002
- added link left_ee_y_axis; visual cylinder length=0.06 radius=0.002
- added link left_ee_z_axis; visual cylinder length=0.06 radius=0.002
- added link left_endeffector; visual sphere radius=0.005
Joints:
- added joint left_ee_x_axis_joint: type fixed, parent left_hand_palm_link, child left_ee_x_axis, origin xyz=0.07 -0.07 0.0 rpy=-1.57 -1.57 0
- added joint left_ee_y_axis_joint: type fixed, parent left_hand_palm_link, child left_ee_y_axis, origin xyz=0.07 -0.07 0.0 rpy=-1.57 -1.57 0
- added joint left_ee_z_axis_joint: type fixed, parent left_hand_palm_link, child left_ee_z_axis, origin xyz=0.07 -0.07 0.0 rpy=-1.57 -1.57 0
- added joint left_endeffector_joint: type fixed, parent left_hand_palm_link, child left_endeffector, origin xyz=0.07 -0.07 0.0 rpy=-1.57 0 0

File: roboverse_data/robots/g1/urdf/g1_mygym_with_world.urdf (robot description, URDF)
Before this commit: robot g1_29dof_with_hand_rev_1_0, 62 links, 61 joints
Links:
- removed link world
Joints:
- removed joint base_to_world

Commit message: add dagger to separate. fix training fingers

File: roboverse_data/robots/g1/urdf/g1_mygym.urdf (robot description, URDF)
Before this commit: robot g1_29dof_with_hand_rev_1_0, 61 links, 60 joints
Joints:
- joint ee_x_axis_joint: origin xyz=0.07 0.07 0.0 rpy=-1.57 -1.57 0 -> xyz=0.07 0.05 0.0 rpy=-1.57 -1.57 0
- joint ee_y_axis_joint: origin xyz=0.07 0.07 0.0 rpy=-1.57 -1.57 0 -> xyz=0.07 0.05 0.0 rpy=-1.57 -1.57 0
- joint ee_z_axis_joint: origin xyz=0.07 0.07 0.0 rpy=-1.57 -1.57 0 -> xyz=0.07 0.05 0.0 rpy=-1.57 -1.57 0
- joint endeffector_joint: origin xyz=0.07 0.07 0.0 rpy=1.57 0 0 -> xyz=0.07 0.05 0.0 rpy=1.57 0 0
- joint left_ee_x_axis_joint: origin xyz=0.07 -0.07 0.0 rpy=-1.57 -1.57 0 -> xyz=0.07 -0.05 0.0 rpy=-1.57 -1.57 0
- joint left_ee_y_axis_joint: origin xyz=0.07 -0.07 0.0 rpy=-1.57 -1.57 0 -> xyz=0.07 -0.05 0.0 rpy=-1.57 -1.57 0
- joint left_ee_z_axis_joint: origin xyz=0.07 -0.07 0.0 rpy=-1.57 -1.57 0 -> xyz=0.07 -0.05 0.0 rpy=-1.57 -1.57 0
- joint left_endeffector_joint: origin xyz=0.07 -0.07 0.0 rpy=-1.57 0 0 -> xyz=0.07 -0.05 0.0 rpy=-1.57 0 0
