Commit message: add door_opening

File: roboverse_data/assets/humanoidbench/door/door3.urdf (robot description, URDF)
Before this commit: robot wall_with_single_door, 6 links, 5 joints
Links:
- removed link door_handle
- link door: mass 1.0 -> 5.0
Joints:
- removed joint door_handle_fixed
- joint door_hinge: limit lower=-1.5708 upper=1.5708 effort=1.0 velocity=5.0 -> lower=-1.5708 upper=1.5708 effort=10.0 velocity=2.0; origin xyz=-0.5 0 0.0 -> xyz=-0.5 0 1.05 rpy=0 0 0
- joint wall_left_fixed: origin (none) -> xyz=0 0 0 rpy=0 0 0
- joint wall_lintel_fixed: origin (none) -> xyz=0 0 0 rpy=0 0 0
- joint wall_right_fixed: origin (none) -> xyz=0 0 0 rpy=0 0 0
