Commit message: cube more up

File: roboverse_data/assets/humanoidbench/door/door.urdf (robot description, URDF)
Before this commit: robot wall_with_single_door, 5 links, 4 joints
Links:
- added link door_handle, mass 0.2; collision box size=0.2 0.02 0.2; visual box size=0.02 0.1 0.02
Joints:
- added joint door_handle_fixed: type fixed, parent door, child door_handle, origin xyz=0 0 0
- joint door_hinge: origin xyz=-0.5 0 1.05 rpy=0 0 0 -> xyz=-0.5 0 0.0
- joint wall_left_fixed: origin xyz=0 0 0 rpy=0 0 0 -> (none)
- joint wall_lintel_fixed: origin xyz=0 0 0 rpy=0 0 0 -> (none)
- joint wall_right_fixed: origin xyz=0 0 0 rpy=0 0 0 -> (none)

Commit message: ready to train stand, door, reach i hope

File: roboverse_data/assets/humanoidbench/door/door.urdf (robot description, URDF)
Before this commit: robot wall_with_single_door, 6 links, 5 joints
Links:
- link door: geometry collision box size=0.57 0.05 1.9; visual box size=0.57 0.05 1.9
- link wall_left: geometry collision box size=2.2 0.05 3.0; visual box size=2.2 0.05 3.0
- link wall_right: geometry collision box size=2.2 0.05 3.0; visual box size=2.2 0.05 3.0
Joints:
- joint door_hinge: origin xyz=-0.5 0 0.0 -> xyz=-0.3 0 0.0

File: roboverse_data/assets/humanoidbench/door/door2.urdf (robot description, URDF)
Before this commit: robot wall_with_single_door, 5 links, 4 joints
Links:
- added link door_handle, mass 0.2; collision box size=0.2 0.02 0.2; visual box size=0.02 0.1 0.02
- link door: mass 5.0 -> 1.0
Joints:
- added joint door_handle_fixed: type fixed, parent door, child door_handle, origin xyz=0 0 0
- joint door_hinge: limit lower=-1.5708 upper=1.5708 effort=10.0 velocity=2.0 -> lower=-1.5708 upper=1.5708 effort=1.0 velocity=5.0; origin xyz=-0.5 0 1.05 rpy=0 0 0 -> xyz=-0.5 0 0.0
- joint wall_left_fixed: origin xyz=0 0 0 rpy=0 0 0 -> (none)
- joint wall_lintel_fixed: origin xyz=0 0 0 rpy=0 0 0 -> (none)
- joint wall_right_fixed: origin xyz=0 0 0 rpy=0 0 0 -> (none)

Commit message: fix get_states in genesis

File: roboverse_data/assets/humanoidbench/door/door.urdf (robot description, URDF)
Before this commit: robot wall_with_single_door, 6 links, 5 joints
Links:
- added link door_handle_stem, mass 0.08; collision box size=0.02 0.1 0.02; visual box size=0.02 0.1 0.02
- link door_handle: mass 0.2 -> 0.12; geometry collision box size=0.1 0.02 0.02; visual box size=0.1 0.02 0.02
Joints:
- added joint door_handle_parts_fixed: type fixed, parent door_handle, child door_handle_stem, origin xyz=0.05 -0.04 -1.0 rpy=0 0 0
- joint door_handle_fixed: origin xyz=0 0 0 -> xyz=0.5 0.06 -0. rpy=0 0 0
- joint door_hinge: origin xyz=-0.3 0 0.0 -> xyz=-0.3 0 1.05

Commit message: door train with simple robot

File: roboverse_data/assets/humanoidbench/door/door.urdf (robot description, URDF)
Before this commit: robot wall_with_single_door, 7 links, 6 joints
Links:
- added link rot_root, mass 0.0
- link door_handle: geometry collision box size=0.10 0.02 0.02; visual box size=0.02 0.1 0.02
- link door_handle_stem: geometry collision box size=0.02 0.20 0.02; visual box size=0.2 0.020 0.02
Joints:
- added joint rot_root_to_wall_base: type fixed, parent rot_root, child wall_base, origin xyz=0 0 0 rpy=0 0 1.57079632679
- joint door_handle_fixed: origin xyz=0.5 0.06 -0. rpy=0 0 0 -> xyz=0.46 0.21 1.0 rpy=0 0 -1.57079632679
- joint door_handle_parts_fixed: origin xyz=0.05 -0.04 -1.0 rpy=0 0 0 -> xyz=0.09 0.05 0.0 rpy=0 0 0
- joint door_hinge: origin xyz=-0.3 0 1.05 -> xyz=-0.3 0 0.0

Commit message: new walk

File: roboverse_data/assets/humanoidbench/door/door.urdf (robot description, URDF)
Before this commit: robot wall_with_single_door, 8 links, 7 joints
Links:
- link door_handle: geometry collision box size=0.02 0.1 0.02; visual box size=0.02 0.1 0.02
- link door_handle_stem: geometry collision box size=0.2 0.020 0.02; visual box size=0.2 0.020 0.02

Commit message: add eval callback

File: roboverse_data/assets/humanoidbench/door/door.urdf (robot description, URDF)
Before this commit: robot wall_with_single_door, 8 links, 7 joints
Links:
- link door: geometry collision box size=0.97 0.05 1.9; visual box size=0.97 0.05 1.9
Joints:
- joint door_handle_fixed: origin xyz=0.46 0.21 1.0 rpy=0 0 -1.57079632679 -> xyz=0.8 0.21 1.0 rpy=0 0 -1.57079632679

File: roboverse_data/robots/g1/urdf/g1_mygym_for_reach.urdf (robot description, URDF)
Before this commit: robot g1_29dof_with_hand_rev_1_0, 54 links, 53 joints
Links:
- link right_wrist_roll_link: geometry collision mesh filename=meshes/right_wrist_roll_link.STL; visual mesh filename=meshes/right_wrist_roll_link.STL
Joints:
- joint right_elbow_joint: limit lower=-1.0472 upper=2.0944 effort=100 velocity=37 -> lower=-1.0472 upper=2.0944 effort=200 velocity=37
- joint right_shoulder_pitch_joint: limit lower=-3.0892 upper=2.6704 effort=50 velocity=37 -> lower=-3.0892 upper=2.6704 effort=200 velocity=37
- joint right_shoulder_roll_joint: limit lower=-2.2515 upper=1.5882 effort=100 velocity=37 -> lower=-2.2515 upper=1.5882 effort=200 velocity=37
- joint right_shoulder_yaw_joint: limit lower=-2.618 upper=2.618 effort=100 velocity=37 -> lower=-2.618 upper=2.618 effort=200 velocity=37
- joint right_wrist_pitch_joint: limit lower=-1.614429558 upper=1.614429558 effort=100 velocity=22 -> lower=-1.614429558 upper=1.614429558 effort=200 velocity=22
- joint right_wrist_roll_joint: limit lower=-1.972222054 upper=1.972222054 effort=100 velocity=37 -> lower=-1.972222054 upper=1.972222054 effort=200 velocity=37
- joint right_wrist_yaw_joint: limit lower=-1.614429558 upper=1.614429558 effort=100 velocity=22 -> lower=-1.614429558 upper=1.614429558 effort=200 velocity=22
- joint waist_pitch_joint: limit lower=-0.52 upper=0.52 effort=50 velocity=37 -> lower=-0.52 upper=0.52 effort=500 velocity=37
- joint waist_roll_joint: limit lower=-0.52 upper=0.52 effort=50 velocity=37 -> lower=-0.52 upper=0.52 effort=500 velocity=37
- joint waist_yaw_joint: limit lower=-2.618 upper=2.618 effort=88 velocity=32 -> lower=-2.618 upper=2.618 effort=500 velocity=32

Commit message: zaloha doorman

File: roboverse_data/assets/humanoidbench/door/door.urdf (robot description, URDF)
Before this commit: robot wall_with_single_door, 8 links, 7 joints
Links:
- link door: mass 1.0 -> 20.0
- link door_handle: mass 0.12 -> 0.5; geometry collision box size=0.02 0.15 0.02; visual box size=0.02 0.15 0.02
- link door_handle_stem: mass 0.08 -> 0.5; geometry collision box size=0.1 0.020 0.02; visual box size=0.1 0.020 0.02
- link wall_left: geometry collision box size=2.1 0.05 3.0; visual box size=2.2 0.05 3.0
Joints:
- removed joint door_handle_fixed
- removed joint door_handle_parts_fixed
- added joint door_handle_joint: type revolute, parent door, child door_handle_stem, origin xyz=0.85 0.21 1.0 rpy=0 0 -1.57079632679, axis 1 0 0, limit lower=0.0 upper=0.8 effort=5.0 velocity=10.0
- added joint stem_to_handle_fixed: type fixed, parent door_handle_stem, child door_handle, origin xyz=0.09 0.05 0.0 rpy=3.14 0 0
- joint door_hinge: limit lower=-1.5708 upper=1.5708 effort=1.0 velocity=5.0 -> lower=-1.5708 upper=0.0 effort=1000.0 velocity=5.0
