Commit message: working sapien3 reach

File: roboverse_data/assets/humanoidbench/cube/cube_2/cube_2.urdf (robot description, URDF)
Before this commit: robot cube_2, 1 links, 0 joints
Links:
- added link base_link
Joints:
- added joint cube_2_fixed_joint: type fixed, parent base_link, child cube_2_link

File: roboverse_data/assets/humanoidbench/table/table.urdf (robot description, URDF)
Before this commit: robot table, 1 links, 0 joints
Links:
- link base_link: mass 0.25 -> 10.0; geometry collision box size=0.05 0.05 0.75; collision box size=0.05 0.05 0.75

Commit message: separate reach only pose and reach pose and orientation

File: roboverse_data/assets/humanoidbench/cube/cube_2/cube_2.urdf (robot description, URDF)
Before this commit: robot cube_2, 2 links, 1 joints
Links:
- link cube_2_link: geometry visual box size=0.05 0.05 0.05

File: roboverse_data/robots/g1/urdf/g1_mygym.urdf (robot description, URDF)
Before this commit: robot g1_29dof_with_hand_rev_1_0, 54 links, 53 joints
Joints:
- joint pelvis_contour_joint: child pelvis -> pelvis_contour_link; parent pelvis_contour_link -> pelvis

Commit message: g1_stand_RL ready to train

File: roboverse_data/assets/humanoidbench/cube/cube_2/cube_2.urdf (robot description, URDF)
Before this commit: robot cube_2, 2 links, 1 joints
Links:
- link cube_2_link: geometry collision box size=0.05 0.05 0.05; visual box size=0.05 0.05 0.05

Commit message: add option external force

File: roboverse_data/assets/humanoidbench/cube/cube_2/cube_2.urdf (robot description, URDF)
Before this commit: robot cube_2, 2 links, 1 joints
Links:
- removed link base_link
Joints:
- removed joint cube_2_fixed_joint

File: roboverse_data/assets/humanoidbench/table/urdf/table.urdf (robot description, URDF)
Before this commit: robot table, 2 links, 1 joints
Links:
- removed link dummy_base
Joints:
- removed joint root_joint
