Commit message: Add Genesis Gaussian splat support

File: roboverse_data/assets/humanoidbench/chairs/chair1/foldable_chair_debug.urdf (robot description, URDF)
Before this commit: robot foldable_chair_gen, 13 links, 12 joints
Links:
- link base_link: geometry collision mesh filename=mesh/foldable_chair.stl scale=0.02 0.02 0.02; visual mesh filename=mesh/foldable_chair.stl scale=0.02 0.02 0.02
- link debug_com: geometry 
- link debug_foot_0: geometry 
- link debug_foot_1: geometry 
- link debug_foot_2: geometry 
- link debug_foot_3: geometry 
- link debug_top_center: geometry 
- link debug_vec: geometry 
- link link_2: geometry 
- link target_hand_left: geometry 
- link target_hand_right: geometry 

File: roboverse_data/robots/g1/urdf/g1_mygym_rotslide_simple.urdf (robot description, URDF)
Before this commit: robot g1_29dof_with_hand_rev_1_0, 65 links, 64 joints
Links:
- link ee_x_axis: geometry 
- link ee_y_axis: geometry 
- link ee_z_axis: geometry 
- link endeffector: geometry 
- link left_ee_x_axis: geometry 
- link left_ee_y_axis: geometry 
- link left_ee_z_axis: geometry 
- link left_endeffector: geometry 
